File: Chassis/Chassis.kicad_pcb (KiCad board)
At the start: 4 copper layers, 80 x 80.1 mm, 75 parts, among them IC1 LV2862YDDCR, IC2 RT6285GSP, J1 FR_JST, J10 IN_XT30, J11 SWD_IN, J12 Conn_01x08_Pin, J13 GIM1_JST, J14 GIM2_JST, J15 GIM1_XT30, J16 GIM2_XT30, J17 SWD_OUT, J18 CHA_XT30, J19 SHOO_XT30, J2 BR_JST, J20 GIM_XT30, J21 OUT_JST, J22 5V_XT30, J23 UART_IN, J24 UART_Out, J25 REF_IN, J26 REF_OUT, J27 CAN2_IN, J28 CAN2_OUT, J3 FL_JST, J4 BL_JST, J5 FR_XT30, J6 BR_XT30, J7 FL_XT30, J8 BL_XT30, J9 IN_JST

Commit message: Finish watchdog schematic
idk if it works lol
Parts:
- added C10: 22µF, Capacitor_SMD:C_0805_2012Metric_Pad1.18x1.45mm_HandSolder, F.Cu at (180.3, 58.3)
- added C11: 100nF, Capacitor_SMD:C_0603_1608Metric_Pad1.08x0.95mm_HandSolder, F.Cu at (175.7, 47.0)
- added C12: 22µF, Capacitor_SMD:C_0805_2012Metric_Pad1.18x1.45mm_HandSolder, F.Cu at (165.0, 58.3)
- added C13: 100nF, Capacitor_SMD:C_0603_1608Metric_Pad1.08x0.95mm_HandSolder, F.Cu at (160.4, 47.0)
- added C14: 22µF, Capacitor_SMD:C_0805_2012Metric_Pad1.18x1.45mm_HandSolder, F.Cu at (149.8, 58.3)
- added C15: 100nF, Capacitor_SMD:C_0603_1608Metric_Pad1.08x0.95mm_HandSolder, F.Cu at (145.2, 47.0)
- added C16: 100nF, Capacitor_SMD:C_0603_1608Metric_Pad1.08x0.95mm_HandSolder, F.Cu at (180.9, 71.6)
- added C17: 100nF, Capacitor_SMD:C_0603_1608Metric_Pad1.08x0.95mm_HandSolder, F.Cu at (175.7, 49.5)
- added C18: 100nF, Capacitor_SMD:C_0603_1608Metric_Pad1.08x0.95mm_HandSolder, F.Cu at (160.4, 49.5)
- added C19: 100nF, Capacitor_SMD:C_0603_1608Metric_Pad1.08x0.95mm_HandSolder, F.Cu at (145.2, 49.5)
- added C20: 10µF, Capacitor_SMD:C_0603_1608Metric_Pad1.08x0.95mm_HandSolder, F.Cu at (175.7, 52.0)
- added C21: 10µF, Capacitor_SMD:C_0603_1608Metric_Pad1.08x0.95mm_HandSolder, F.Cu at (160.4, 52.0)
- added C22: 10µF, Capacitor_SMD:C_0603_1608Metric_Pad1.08x0.95mm_HandSolder, F.Cu at (145.2, 52.0)
- added D11: BAS21,235, Package_TO_SOT_SMD:SOT-23, F.Cu at (180.3, 54.6)
- added D12: BAS21,235, Package_TO_SOT_SMD:SOT-23, F.Cu at (165.1, 54.6)
- added D13: BAS21,235, Package_TO_SOT_SMD:SOT-23, F.Cu at (149.8, 54.6)
- added IC3: TPS1HC100BQPWPRQ1, Robomaster_ICs:SOP65P640X120-15N, F.Cu at (182.3, 49.1)
- added IC4: TPS1HC100BQPWPRQ1, Robomaster_ICs:SOP65P640X120-15N, F.Cu at (167.1, 49.1)
- added IC5: TPS1HC100BQPWPRQ1, Robomaster_ICs:SOP65P640X120-15N, F.Cu at (151.8, 49.1)
- added IC6: MIC826RYMT-TR, Robomaster_ICs:SON50P160X160X60-7N-D, F.Cu at (180.7, 77.2)
- added J29: Conn_01x04_Pin, Connector_JST:JST_GH_BM04B-GHS-TBT_1x04-1MP_P1.25mm_Vertical, F.Cu at (163.5, 74.2)
- added J30: Conn_01x02_Pin, Connector_JST:JST_GH_BM02B-GHS-TBT_1x02-1MP_P1.25mm_Vertical, F.Cu at (174.8, 74.2)
- added J32: Conn_01x02, Connector_JST:JST_GH_BM02B-GHS-TBT_1x02-1MP_P1.25mm_Vertical, F.Cu at (162.3, 81.8)
- added R12: 5kΩ, Resistor_SMD:R_0603_1608Metric_Pad0.98x0.95mm_HandSolder, F.Cu at (175.7, 54.5)
- added R13: 5kΩ, Resistor_SMD:R_0603_1608Metric_Pad0.98x0.95mm_HandSolder, F.Cu at (175.7, 57.0)
- added R14: 1kΩ, Resistor_SMD:R_0603_1608Metric_Pad0.98x0.95mm_HandSolder, F.Cu at (175.7, 59.5)
- added R15: 5kΩ, Resistor_SMD:R_0603_1608Metric_Pad0.98x0.95mm_HandSolder, F.Cu at (175.7, 62.1)
- added R16: 18kΩ, Resistor_SMD:R_0603_1608Metric_Pad0.98x0.95mm_HandSolder, F.Cu at (175.7, 64.6)
- added R17: 1kΩ, Resistor_SMD:R_0603_1608Metric_Pad0.98x0.95mm_HandSolder, F.Cu at (175.7, 67.1)
- added R18: 5kΩ, Resistor_SMD:R_0603_1608Metric_Pad0.98x0.95mm_HandSolder, F.Cu at (160.4, 54.5)
- added R19: 5kΩ, Resistor_SMD:R_0603_1608Metric_Pad0.98x0.95mm_HandSolder, F.Cu at (160.4, 57.0)
- added R20: 1kΩ, Resistor_SMD:R_0603_1608Metric_Pad0.98x0.95mm_HandSolder, F.Cu at (160.4, 59.5)
- added R21: 5kΩ, Resistor_SMD:R_0603_1608Metric_Pad0.98x0.95mm_HandSolder, F.Cu at (160.4, 62.1)
- added R22: 18kΩ, Resistor_SMD:R_0603_1608Metric_Pad0.98x0.95mm_HandSolder, F.Cu at (160.4, 64.6)
- added R23: 1kΩ, Resistor_SMD:R_0603_1608Metric_Pad0.98x0.95mm_HandSolder, F.Cu at (160.4, 67.1)
- added R24: 5kΩ, Resistor_SMD:R_0603_1608Metric_Pad0.98x0.95mm_HandSolder, F.Cu at (145.2, 54.5)
- added R25: 5kΩ, Resistor_SMD:R_0603_1608Metric_Pad0.98x0.95mm_HandSolder, F.Cu at (145.2, 57.0)
- added R26: 1kΩ, Resistor_SMD:R_0603_1608Metric_Pad0.98x0.95mm_HandSolder, F.Cu at (145.2, 59.5)
- added R27: 5kΩ, Resistor_SMD:R_0603_1608Metric_Pad0.98x0.95mm_HandSolder, F.Cu at (145.2, 62.1)
- added R28: 18kΩ, Resistor_SMD:R_0603_1608Metric_Pad0.98x0.95mm_HandSolder, F.Cu at (145.2, 64.6)
- added R29: 1kΩ, Resistor_SMD:R_0603_1608Metric_Pad0.98x0.95mm_HandSolder, F.Cu at (145.2, 67.1)
- added R30: 1kΩ, Resistor_SMD:R_0603_1608Metric_Pad0.98x0.95mm_HandSolder, F.Cu at (180.9, 74.1)
- F1: value Fuse -> 2A
Connections:
- C2 pad 1: Mini_PC -> +24V
- C7 pad 1: Mini_PC -> +24V
- C8 pad 1: Mini_PC -> +24V
- D10 pad 1: Net-(D10-K) -> +24V
- F1 pad 1: Mini_PC -> Mini PC
- F1 pad 2: Net-(D10-K) -> +24V
- IC1 pad 5: Mini_PC -> +24V
- IC2 pad 7: Mini_PC -> +24V
- J10 pad 2: Mini_PC -> Mini PC
- J12 pad 5: +24V_Shooter -> +24V Shooter OUT
- J12 pad 6: +24V_Gimbal -> +24V Gimbal OUT
- J15 pad 2: +24V_Gimbal -> +24V Gimbal OUT
- J16 pad 2: +24V_Gimbal -> +24V Gimbal OUT
- J18 pad 2: +24V_Chassis -> +24V Chassis IN
- J19 pad 2: +24V_Shooter -> +24V Shooter IN
- J20 pad 2: +24V_Gimbal -> +24V Gimbal IN
- J5 pad 2: +24V_Chassis -> +24V Chassis OUT
- J6 pad 2: +24V_Chassis -> +24V Chassis OUT
- J7 pad 2: +24V_Chassis -> +24V Chassis OUT
- J8 pad 2: +24V_Chassis -> +24V Chassis OUT
- R10 pad 2: +24V_Shooter -> +24V Shooter OUT
- R11 pad 2: Mini_PC -> +24V
- R2 pad 2: Mini_PC -> +24V
- R8 pad 2: +24V_Gimbal -> +24V Gimbal OUT
- R9 pad 2: +24V_Chassis -> +24V Chassis OUT
- TP3 pad 1: Mini_PC -> +24V
Routing:
- net (no net): track 0.00 -> 19.5 mm, vias 0 -> 1
- net +24V: track 0.00 -> 18.6 mm, vias 0 -> 8
- net Mini_PC: track 16.5 -> 0.00 mm, vias 9 -> 0
- net Net-(D10-K): track 10.3 -> 0.00 mm
- net +24V_Shooter: track 6.37 -> 0.00 mm
- net +24V_Gimbal: track 4.85 -> 0.00 mm
- added copper zone on F.Cu, net +24V
- added copper zone on F.Cu, net +24V Chassis OUT
- added copper zone on In2.Cu, net +24V Gimbal IN
- added copper zone on In2.Cu, net +24V Shooter OUT
- added copper zone on F.Cu, net Mini PC
- added copper zone on In2.Cu, net Mini PC
- removed copper zone on F.Cu, net +24V_Chassis
- removed copper zone on In2.Cu, net +24V_Gimbal
- removed copper zone on In2.Cu, net +24V_Shooter
- removed copper zone on F.Cu, net Mini_PC
- removed copper zone on In2.Cu, net Mini_PC
