File: Chassis/Chassis.kicad_sch (KiCad schematic)
At the start: 48 parts, among them J1 FR_JST, J10 IN_XT30, J11 SWD_IN, J12 Conn_01x08_Pin, J13 GIM1_JST, J14 GIM2_JST, J15 GIM1_XT30, J16 GIM2_XT30, J17 SWD_OUT, J18 CHA_XT30, J19 SHOO_XT30, J2 BR_JST, J20 GIM_XT30, J21 OUT_JST, J22 5V_XT30, J23 UART_IN, J24 UART_Out, J25 REF_IN, J26 REF_OUT, J27 CAN2_IN, J28 CAN2_OUT, J3 FL_JST, J4 BL_JST, J5 FR_XT30, J6 BR_XT30, J7 FL_XT30, J8 BL_XT30, J9 IN_JST

Commit message: Add HSS
Other:
- sheet Watchdog ports: added SNS_{Chassis}, SNS_{Gimbal}, SNS_{Shooter}, V_{IN,Chassis}, V_{IN,Gimbal}, V_{IN,Shooter}, V_{OUT,Chassis}, V_{OUT,Gimbal}, V_{OUT,Shooter}, WDI, ~{MR}; removed none
Changed lines of the file:
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@@
       (effects (font (size 1.27 1.27)) (justify left top))
+    )
+    (pin "V_{IN,Shooter}" input (at 238.76 88.9 180)
+      (effects (font (size 1.27 1.27)) (justify left))
+    )
+    (pin "SNS_{Shooter}" output (at 251.46 82.55 90)
+      (effects (font (size 1.27 1.27)) (justify right))
+    )
+    (pin "SNS_{Gimbal}" output (at 254 82.55 90)
+      (effects (font (size 1.27 1.27)) (justify right))
+    )
+    (pin "V_{IN,Gimbal}" input (at 238.76 91.44 180)
+      (effects (font (size 1.27 1.27)) (justify left))
+    )
+    (pin "SNS_{Chassis}" output (at 256.54 82.55 90)
+      (effects (font (size 1.27 1.27)) (justify right))
+    )
+    (pin "V_{IN,Chassis}" input (at 238.76 93.98 180)
+      (effects (font (size 1.27 1.27)) (justify left))
+    )
+    (pin "V_{OUT,Chassis}" output (at 271.78 93.98 0)
+      (effects (font (size 1.27 1.27)) (justify right))
+    )
+    (pin "V_{OUT,Shooter}" output (at 271.78 88.9 0)
+      (effects (font (size 1.27 1.27)) (justify right))
+    )
+    (pin "V_{OUT,Gimbal}" output (at 271.78 91.44 0)
+      (effects (font (size 1.27 1.27)) (justify right))
+    )
+    (pin "WDI" input (at 254 105.41 270)
+      (effects (font (size 1.27 1.27)) (justify left))
+    )
+    (pin "~{MR}" input (at 256.54 105.41 270)
+      (effects (font (size 1.27 1.27)) (justify left))
     )
     (instances

Commit message: Finish watchdog schematic
idk if it works lol
Parts:
- added J29: Conn_01x04_Pin, Connector_JST:JST_GH_BM04B-GHS-TBT_1x04-1MP_P1.25mm_Vertical, symbol Connector:Conn_01x04_Pin
- added J32: Conn_01x02, Connector_JST:JST_GH_BM02B-GHS-TBT_1x02-1MP_P1.25mm_Vertical, symbol Connector_Generic:Conn_01x02
- F1: value Fuse -> 2A
Connections:
- net GND: now also J29.4 (Pin_4), J32.2 (Pin_2)
- net Watchdog/SNS_{Chassis}: now also J29.1 (Pin_1)
- net Watchdog/SNS_{Gimbal}: now also J29.2 (Pin_2)
- net Watchdog/SNS_{Shooter}: now also J29.3 (Pin_3)
- net Watchdog/WDI: now also J32.1 (Pin_1)
- net +24V: now reaches D10.1 (K), F1.2
- net +24V: now also R2.2
- net +24V_Chassis renamed +24V Chassis OUT
- net +24V Chassis OUT: no longer J18.2 (Pin_2)
- net +24V_Gimbal renamed +24V Gimbal OUT
- net +24V Gimbal OUT: no longer J20.2 (Pin_2)
- net +24V_Shooter renamed +24V Shooter OUT
- net +24V Shooter OUT: no longer J19.2 (Pin_2)
- net Mini_PC renamed Mini PC
- net Mini PC: no longer R2.2
- new net +24V Chassis IN: J18.2 (Pin_2)
- new net +24V Gimbal IN: J20.2 (Pin_2)
- new net +24V Shooter IN: J19.2 (Pin_2)
Other:
- sheet Watchdog ports: added none; removed ~{MR}
- moved on the sheet: J13, J14, J15, J16
