File: Chassis/hsswitch.kicad_sch (KiCad schematic)
At the start: 10 parts, among them IC4 TPS1HC100BQPWPRQ1

Commit message: Finish watchdog schematic
idk if it works lol
Parts:
- added C10: 10µF, Capacitor_SMD:C_0603_1608Metric_Pad1.08x0.95mm_HandSolder, symbol Device:C
- added C10: 100nF, Capacitor_SMD:C_0603_1608Metric_Pad1.08x0.95mm_HandSolder, symbol Device:C
- C10: footprint (none) -> Capacitor_SMD:C_0603_1608Metric_Pad1.08x0.95mm_HandSolder
- C11: footprint (none) -> Capacitor_SMD:C_0805_2012Metric_Pad1.18x1.45mm_HandSolder
- R12, R13, R16: footprint (none) -> Resistor_SMD:R_0603_1608Metric_Pad0.98x0.95mm_HandSolder
- R14, R15: footprint (none) -> Resistor_SMD:R_0603_1608Metric_Pad0.98x0.95mm_HandSolder; Manufacturer_Name (none) -> YAGEO; Manufacturer_Part_Number (none) -> RT0603BRE075KL; Mouser Part Number (none) -> 603-RT0603BRE075KL
Connections:
- net GND: now also C10.2, C10.2
- net SNS: now also C10.1
- net V_{IN}: now also C10.1
Other:
- note added: "Bulk capacitance (place in vicinity)"
- note added: "Current sense"
- note added: "EMI protection (place as close as possible)"
- note added: "For reducing current for switching off inductive loads (Flyback kinda)"
- note added: "High-side Switch IC"
- note added: "I_{LIM} = ^{45kΩ•A}/_{1.8kΩ} = 2.5A"
- moved on the sheet: R13, R14, R15
