File: Chassis/watchdog.kicad_sch (KiCad schematic)
At the start: 0 parts

Commit message: Trying to implement the high-side switching for the watchdog
Parts:
- added C10: 100nF, symbol Device:C
- added C11: 22µF, symbol Device:C
- added D11: BAS21,235, Package_TO_SOT_SMD:SOT-23, symbol Device:D
- added IC4: TPS1HC100BQPWPRQ1, Robomaster_ICs:SOP65P640X120-15N, symbol Robomaster_Library:TPS1HC100BQPWPRQ1
- added R12, R13: 1kΩ, symbol Device:R
- added R14, R15: 5kΩ, symbol Device:R
Connections:
- new net: IC4.2 (EN), R15.2
- new net: IC4.3 (DIAG_EN), R14.2
- new net +5V: R14.1
- new net AGND: D11.2 (A), IC4.1 (GND_1), IC4.15 (GND_2), R12.1
- new net EN: R15.1
- new net GND: C10.2, C11.2, D11.1 (K), R12.2, R13.2
- new net SNS: IC4.6 (SNS), R13.1
- new net V_{IN}: C10.1, IC4.12 (VBB_1), IC4.13 (VBB_2)
- new net V_{OUT}: C11.1, IC4.10 (VOUT_2), IC4.9 (VOUT_1)
- no-connect marks 0 -> 5

Commit message: Add HSS
Parts:
- removed C10: 100nF, symbol Device:C
- removed C11: 22µF, symbol Device:C
- removed D11: BAS21,235, Package_TO_SOT_SMD:SOT-23, symbol Device:D
- removed IC4: TPS1HC100BQPWPRQ1, Robomaster_ICs:SOP65P640X120-15N, symbol Robomaster_Library:TPS1HC100BQPWPRQ1
- removed R12, R13: 1kΩ, symbol Device:R
- removed R14, R15: 5kΩ, symbol Device:R
- added C16: 100nF, symbol Device:C
- added IC6: MIC826RYMT-TR, Robomaster_ICs:SON50P160X160X60-7N-D, symbol Robomaster_Library:MIC826RYMT-TR
Connections:
- net +5V: now also C16.1, IC6.6 (VCC)
- net EN: now also IC6.1 (~{RESET})
- net GND: now also C16.2, IC6.2 (GND), IC6.7 (EP)
- new net WDI: IC6.4 (WDI)
- new net ~{MR}: IC6.5 (~{MR})
- no-connect marks 5 -> 1
Other:
- added sheet High-Side Switch (Chassis) (hsswitch.kicad_sch)
- added sheet High-Side Switch (Gimbal) (hsswitch.kicad_sch)
- added sheet High-Side Switch (Shooter) (hsswitch.kicad_sch)

Commit message: Finish watchdog schematic
idk if it works lol
Parts:
- added J30: Conn_01x02_Pin, Connector_JST:JST_GH_BM02B-GHS-TBT_1x02-1MP_P1.25mm_Vertical, symbol Connector:Conn_01x02_Pin
- added R30: 1kΩ, Resistor_SMD:R_0603_1608Metric_Pad0.98x0.95mm_HandSolder, symbol Device:R
- C16: footprint (none) -> Capacitor_SMD:C_0603_1608Metric_Pad1.08x0.95mm_HandSolder
Connections:
- net +5V: now also R30.1
- net GND: now also J30.2 (Pin_2)
- net ~{MR}: no longer names the net of IC6.5 (~{MR})
- net ~{MR}: now also J30.1 (Pin_1), R30.2
Other:
- note added: "High-side switches"
- note added: "Watchdog Timer IC"
- moved on the sheet: C16, IC6
