File: ElectricalDiagram/Turret.kicad_sch (KiCad schematic)
At the start: 25 parts

Commit message: Prepped Electrical Diagram for meeting
Parts:
- removed +19V1, +24V_Gimbal2, +24V_Shooter1, +5V1, GND1: TestPoint, TestPoint:TestPoint_Loop_D1.80mm_Drill1.0mm_Beaded, symbol Connector:TestPoint
- removed +19V_Turret->Orin1, +24V_Feeder1, +24V_Gimbal1, +24V_L_Flywheel1, +24V_R_Flywheel1, +24V_Waterwheel1: Conn_01x02_Pin, Robomaster_ICs:AMASS_XT30U-F_1x02_P5.0mm_Vertical_copy, symbol Connector:Conn_01x02_Pin
- removed 8_Pin_Slipring->Turret1: Conn_01x08_Pin, ICs:CON_1722981108_MOL, symbol Connector:Conn_01x08_Pin
- removed CAN_Feeder1, CAN_Gimbal1, CAN_In1, CAN_In2, CAN_L_Flywheel1, CAN_R_Flywheel1, CAN_Waterwheel1: Conn_01x02_Pin, Connector_JST:JST_GH_BM02B-GHS-TBT_1x02-1MP_P1.25mm_Vertical, symbol Connector:Conn_01x02_Pin
- removed Debug_Orin->Turret1, Debug_Turret->Chassis1, Ref_In1, Ref_Out1, UART_Chassis->Turret1, UART_Turret->Orin1: Conn_01x04_Pin, Connector_JST:JST_GH_BM04B-GHS-TBT_1x04-1MP_P1.25mm_Vertical, symbol Connector:Conn_01x04_Pin
- added H1, H2, H3, H4: MountingHole, symbol Mechanical:MountingHole
- added J1 (x6), J2, J? (x6): Conn_01x02_Pin, symbol Connector:Conn_01x02_Pin
- added J1 (x6): Conn_01x04_Pin, symbol Connector:Conn_01x04_Pin
- added J?: Conn_01x08_Pin, symbol Connector:Conn_01x08_Pin
- added TP1, TP? (x4): TestPoint, symbol Connector:TestPoint
Connections:
- net +19V: now also J?.2 (Pin_2), J?.7 (Pin_7), TP?.1
- net +24V_Gimbal: now also J?.2 (Pin_2), J?.6 (Pin_6), TP?.1
- net +24V_Shooter: now also J?.2 (Pin_2), J?.2 (Pin_2), J?.2 (Pin_2), J?.2 (Pin_2), J?.5 (Pin_5), TP?.1
- net +5V: now also J?.8 (Pin_8), TP?.1
- net 3.3V_Debug: now also J1.4 (Pin_4), J1.4 (Pin_4)
- net 3.3V_UART: now also J1.4 (Pin_4), J1.4 (Pin_4)
- net CANH: now also J1.2 (Pin_2), J1.2 (Pin_2), J1.2 (Pin_2), J1.2 (Pin_2), J2.2 (Pin_2)
- net CANHPitch: now also J1.2 (Pin_2), J1.2 (Pin_2)
- net CANHRef: now also J1.3 (Pin_3), J1.3 (Pin_3)
- net CANL: now also J1.1 (Pin_1), J1.1 (Pin_1), J1.1 (Pin_1), J1.1 (Pin_1), J2.1 (Pin_1)
- net CANLPitch: now also J1.1 (Pin_1), J1.1 (Pin_1)
- net CANLRef: now also J1.2 (Pin_2), J1.2 (Pin_2)
- net GND: now also J1.1 (Pin_1), J1.1 (Pin_1), J1.1 (Pin_1), J1.1 (Pin_1), J1.1 (Pin_1), J1.1 (Pin_1), J?.1 (Pin_1), J?.1 (Pin_1), J?.1 (Pin_1), J?.1 (Pin_1), J?.1 (Pin_1), J?.1 (Pin_1), J?.1 (Pin_1), J?.2 (Pin_2), J?.3 (Pin_3), J?.4 (Pin_4), TP1.1
- net Ref_PWR: now also J1.4 (Pin_4), J1.4 (Pin_4)
- net SWCLK: now also J1.3 (Pin_3), J1.3 (Pin_3)
- net SWDIO: now also J1.2 (Pin_2), J1.2 (Pin_2)
- net UART_RX: now also J1.3 (Pin_3), J1.3 (Pin_3)
- net UART_TX: now also J1.2 (Pin_2), J1.2 (Pin_2)
Other:
- note added: "Mounting Holes"
